File: ledmatrix-module.sch (KiCad schematic (older format))
At the start: 3 parts

Commit message: dual matrix with 2x2 interconnects
Parts:
- R1: renamed from R?; footprint (none) -> footprints:0603_HAND
- U1: renamed from U?; footprint (none) -> footprints:LEDMATRIX_1588BS
- U2: renamed from U?; footprint (none) -> SMD_Packages:SO-16-N
Changed lines of the file:
@@
 LIBS:ledmatrix
 LIBS:misc_logic
-LIBS:ledmatrix-dual-cache
+LIBS:ledmatrix-cache
 EELAYER 25 0
 EELAYER END
 $Descr A4 11693 8268
 encoding utf-8
-Sheet 2 5
+Sheet 2 4
 Title ""
 Date ""
@@
 $EndDescr
 $Comp
-L 1588BS U?
+L 1588BS U1
 U 1 1 59AA78F5
 P 6550 2750
-F 0 "U?" H 6550 2750 60  0000 C CNN
+AR Path="/59AA789F/59AA78F5" Ref="U1"  Part="1"
+AR Path="/59AABAB3/59AA78F5" Ref="U3"  Part="1"
+AR Path="/59AB26B1/59AA78F5" Ref="U6"  Part="1"
+F 0 "U1" H 6550 2750 60  0000 C CNN
 F 1 "1588BS" H 6550 2350 60  0000 C CNN
-F 2 "" H 6650 2600 60  0001 C CNN
+F 2 "footprints:LEDMATRIX_1588BS" H 6650 2600 60  0001 C CNN
 F 3 "" H 6650 2600 60  0001 C CNN
 	1    6550 2750
@@
 ROW_8
 $Comp
-L STP08DP05 U?
+L STP08DP05 U2
 U 1 1 59AA7ABF
 P 7800 2750
-F 0 "U?" H 7800 2750 60  0000 C CNN
+AR Path="/59AA789F/59AA7ABF" Ref="U2"  Part="1"
+AR Path="/59AABAB3/59AA7ABF" Ref="U4"  Part="1"
+AR Path="/59AB26B1/59AA7ABF" Ref="U7"  Part="1"
+F 0 "U2" H 7800 2750 60  0000 C CNN
 F 1 "STP08DP05" H 7800 2250 60  0000 C CNN
-F 2 "" H 8000 2500 60  0001 C CNN
+F 2 "SMD_Packages:SO-16-N" H 8000 2500 60  0001 C CNN
 F 3 "" H 8000 2500 60  0001 C CNN
 	1    7800 2750
@@
 	5850 3100 6000 3100
 $Comp
-L R_Small R?
+L R_Small R1
 U 1 1 59AA7F03
 P 9150 2900
-F 0 "R?" H 9180 2920 50  0000 L CNN
+AR Path="/59AA789F/59AA7F03" Ref="R1"  Part="1"
+AR Path="/59AABAB3/59AA7F03" Ref="R2"  Part="1"
+AR Path="/59AB26B1/59AA7F03" Ref="R11"  Part="1"
+F 0 "R1" H 9180 2920 50  0000 L CNN
 F 1 "1k" H 9180 2860 50  0000 L CNN
-F 2 "" H 9150 2900 50  0001 C CNN
+F 2 "footprints:0603_HAND" H 9150 2900 50  0001 C CNN
 F 3 "" H 9150 2900 50  0001 C CNN
 	1    9150 2900

Commit message: fix matrix module order
Changed lines of the file:
@@
 AR Path="/59AABAB3/59AA78F5" Ref="U3"  Part="1"
 AR Path="/59AB26B1/59AA78F5" Ref="U6"  Part="1"
-F 0 "U1" H 6550 2750 60  0000 C CNN
+F 0 "U3" H 6550 2750 60  0000 C CNN
 F 1 "1588BS" H 6550 2350 60  0000 C CNN
 F 2 "footprints:LEDMATRIX_1588BS" H 6650 2600 60  0001 C CNN
@@
 AR Path="/59AABAB3/59AA7ABF" Ref="U4"  Part="1"
 AR Path="/59AB26B1/59AA7ABF" Ref="U7"  Part="1"
-F 0 "U2" H 7800 2750 60  0000 C CNN
+F 0 "U4" H 7800 2750 60  0000 C CNN
 F 1 "STP08DP05" H 7800 2250 60  0000 C CNN
 F 2 "SMD_Packages:SO-16-N" H 8000 2500 60  0001 C CNN
@@
 AR Path="/59AABAB3/59AA7F03" Ref="R2"  Part="1"
 AR Path="/59AB26B1/59AA7F03" Ref="R11"  Part="1"
-F 0 "R1" H 9180 2920 50  0000 L CNN
+F 0 "R2" H 9180 2920 50  0000 L CNN
 F 1 "1k" H 9180 2860 50  0000 L CNN
 F 2 "footprints:0603_HAND" H 9150 2900 50  0001 C CNN

Commit message: save schematic changes
Changed lines of the file:
@@
 AR Path="/59AABAB3/59AA78F5" Ref="U3"  Part="1"
 AR Path="/59AB26B1/59AA78F5" Ref="U6"  Part="1"
-F 0 "U3" H 6550 2750 60  0000 C CNN
+F 0 "U1" H 6550 2750 60  0000 C CNN
 F 1 "1588BS" H 6550 2350 60  0000 C CNN
 F 2 "footprints:LEDMATRIX_1588BS" H 6650 2600 60  0001 C CNN
@@
 AR Path="/59AABAB3/59AA7ABF" Ref="U4"  Part="1"
 AR Path="/59AB26B1/59AA7ABF" Ref="U7"  Part="1"
-F 0 "U4" H 7800 2750 60  0000 C CNN
+F 0 "U2" H 7800 2750 60  0000 C CNN
 F 1 "STP08DP05" H 7800 2250 60  0000 C CNN
 F 2 "SMD_Packages:SO-16-N" H 8000 2500 60  0001 C CNN
@@
 AR Path="/59AABAB3/59AA7F03" Ref="R2"  Part="1"
 AR Path="/59AB26B1/59AA7F03" Ref="R11"  Part="1"
-F 0 "R2" H 9180 2920 50  0000 L CNN
+F 0 "R1" H 9180 2920 50  0000 L CNN
 F 1 "1k" H 9180 2860 50  0000 L CNN
 F 2 "footprints:0603_HAND" H 9150 2900 50  0001 C CNN

Commit message: add bypassing to schematic
Parts:
- added C2: 1u, footprints:0603_HAND, symbol C_Small
Connections:
- net GND: now also C2.2
- net VCC: now also C2.1
Changed lines of the file:
@@
 $Descr A4 11693 8268
 encoding utf-8
-Sheet 2 4
+Sheet 3 4
 Title ""
 Date ""
@@
 	1    0    0    -1
 $EndComp
-Text HLabel 8500 2400 2    60   Input ~ 0
+Text HLabel 8800 2200 2    60   Input ~ 0
 VCC
-Text HLabel 8500 2500 2    60   Input ~ 0
+Text HLabel 8800 2500 2    60   Input ~ 0
 GND
 Text HLabel 8500 2600 2    60   Input ~ 0
@@
 	7100 3100 7200 3100
 Wire Wire Line
-	8400 2400 8500 2400
+	8500 2400 8400 2400
 Wire Wire Line
-	8500 2500 8400 2500
+	8400 2500 8800 2500
 Wire Wire Line
 	8400 2600 8500 2600
@@
 Wire Wire Line
 	9250 2900 9350 2900
+$Comp
+L C_Small C2
+U 1 1 59AC0BD1
+P 8650 2350
+AR Path="/59AA789F/59AC0BD1" Ref="C2"  Part="1"
+AR Path="/59AABAB3/59AC0BD1" Ref="C3"  Part="1"
+F 0 "C2" H 8660 2420 50  0000 L CNN
+F 1 "1u" H 8660 2270 50  0000 L CNN
+F 2 "footprints:0603_HAND" H 8650 2350 50  0001 C CNN
+F 3 "" H 8650 2350 50  0001 C CNN
+	1    8650 2350
+	1    0    0    -1
+$EndComp
+Wire Wire Line
+	8650 2500 8650 2450
+Connection ~ 8650 2500
+Wire Wire Line
+	8500 2200 8500 2400
+Wire Wire Line
+	8500 2200 8800 2200
+Wire Wire Line
+	8650 2250 8650 2200
+Connection ~ 8650 2200
 $EndSCHEMATC

Commit message: fully connected PCB
Changed lines of the file:
@@
 AR Path="/59AABAB3/59AA78F5" Ref="U3"  Part="1"
 AR Path="/59AB26B1/59AA78F5" Ref="U6"  Part="1"
-F 0 "U1" H 6550 2750 60  0000 C CNN
+F 0 "U3" H 6550 2750 60  0000 C CNN
 F 1 "1588BS" H 6550 2350 60  0000 C CNN
 F 2 "footprints:LEDMATRIX_1588BS" H 6650 2600 60  0001 C CNN
@@
 AR Path="/59AABAB3/59AA7ABF" Ref="U4"  Part="1"
 AR Path="/59AB26B1/59AA7ABF" Ref="U7"  Part="1"
-F 0 "U2" H 7800 2750 60  0000 C CNN
+F 0 "U4" H 7800 2750 60  0000 C CNN
 F 1 "STP08DP05" H 7800 2250 60  0000 C CNN
 F 2 "SMD_Packages:SO-16-N" H 8000 2500 60  0001 C CNN
@@
 AR Path="/59AABAB3/59AA7F03" Ref="R2"  Part="1"
 AR Path="/59AB26B1/59AA7F03" Ref="R11"  Part="1"
-F 0 "R1" H 9180 2920 50  0000 L CNN
+F 0 "R2" H 9180 2920 50  0000 L CNN
 F 1 "1k" H 9180 2860 50  0000 L CNN
 F 2 "footprints:0603_HAND" H 9150 2900 50  0001 C CNN
@@
 AR Path="/59AA789F/59AC0BD1" Ref="C2"  Part="1"
 AR Path="/59AABAB3/59AC0BD1" Ref="C3"  Part="1"
-F 0 "C2" H 8660 2420 50  0000 L CNN
+F 0 "C3" H 8660 2420 50  0000 L CNN
 F 1 "1u" H 8660 2270 50  0000 L CNN
 F 2 "footprints:0603_HAND" H 8650 2350 50  0001 C CNN
